Commit message: Add files via upload

File: vehicle_description/urdf/turbopi/turbopi.urdf (robot description, URDF)
Before this commit: robot prototype_one, 10 links, 9 joints
Links:
- removed link prototype_one_back_left_wheel_link
- removed link prototype_one_back_right_wheel_link
- removed link prototype_one_base_footprint
- removed link prototype_one_base_link
- removed link prototype_one_front_left_wheel_link
- removed link prototype_one_front_right_wheel_link
- added link turbopi_back_left_wheel_link, mass 5; collision cylinder length=0.03 radius=0.05; visual cylinder length=0.03 radius=0.05
- added link turbopi_back_right_wheel_link, mass 5; collision cylinder length=0.03 radius=0.05; visual cylinder length=0.03 radius=0.05
- added link turbopi_base_footprint; visual box size=0.001 0.001 0.001
- added link turbopi_base_link, mass 125.0; collision box size=0.4 0.3 0.15; visual box size=0.4 0.3 0.15
- added link turbopi_front_left_wheel_link, mass 5; collision cylinder length=0.03 radius=0.05; visual cylinder length=0.03 radius=0.05
- added link turbopi_front_right_wheel_link, mass 6.5; collision cylinder length=0.087 radius=0.127; visual mesh filename=package://hydra_one_description/models/hydra_one/meshes/whe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
Joints:
- removed joint hydra_one_base_footprint_joint
- removed joint prototype_one_back_left_wheel_joint
- removed joint prototype_one_back_right_wheel_joint
- removed joint prototype_one_front_left_wheel_joint
- removed joint prototype_one_front_right_wheel_joint
- added joint turbopi_back_left_wheel_joint: type continuous, parent turbopi_base_link, child turbopi_back_left_wheel_link, origin xyz=-0.175 0.1645 -0.05 rpy=0 0 0, axis 0 1 0, limit effort=100 velocity=100
- added joint turbopi_back_right_wheel_joint: type continuous, parent turbopi_base_link, child turbopi_back_right_wheel_link, origin xyz=-0.175 -0.1645 -0.05 rpy=0 0 0, axis 0 1 0, limit effort=100 velocity=100
- added joint turbopi_base_footprint_joint: type fixed, parent turbopi_base_footprint, child turbopi_base_link, origin xyz=0 0 0.127 rpy=0 0 0
- added joint turbopi_front_left_wheel_joint: type continuous, parent turbopi_base_link, child turbopi_front_left_wheel_link, origin xyz=0.175 0.1645 -0.05 rpy=0 0 0, axis 0 1 0, limit effort=100 velocity=100
- added joint turbopi_front_right_wheel_joint: type continuous, parent turbopi_base_link, child turbopi_front_right_wheel_link, origin xyz=0.175 -0.1645 -0.05 rpy=0 0 0, axis 0 1 0, limit effort=100 velocity=100
- joint cente-0.05r_laser_joint: parent prototype_one_base_link -> turbopi_base_link
- joint front_depth_sensor_joint: parent prototype_one_base_link -> turbopi_base_link
- joint front_lower_camera_joint: parent prototype_one_base_link -> turbopi_base_link
